File: samn/samn_7.sch (KiCad schematic (older format))
At the start: 31 parts, among them J1 Conn_01x06_Female, J10 Conn_01x06_Female, J11 Conn_01x02, J12 Conn_01x04, J2 Conn_01x02, J3 Conn_01x06_Female, J4 Conn_02x03_Male_ICSP, J5 Conn_01x03, J6 Conn_01x06, J7 Conn_01x06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

Commit message: staring v8 of samn
Parts:
- U2: symbol MCU_Microchip_ATmega:ATmega328PB-AU -> samn_7-rescue:ATmega328PB-AU-MCU_Microchip_ATmega
Changed lines of the file:
@@
 EESchema Schematic File Version 4
-LIBS:samn_small-cache
-EELAYER 29 0
+EELAYER 30 0
 EELAYER END
 $Descr A4 11693 8268
@@
 Connection ~ 8400 3850
 $Comp
-L MCU_Microchip_ATmega:ATmega328PB-AU U2
+L samn_7-rescue:ATmega328PB-AU-MCU_Microchip_ATmega U2
 U 1 1 5C1F8278
 P 7700 3650
